Commit message: fixed gazebo launch file and added color to robot, improved camera

File: install/dofbot_description/share/dofbot_description/urdf/new_cr5.xacro (robot description, xacro)
@@ -6,4 +6,17 @@
 <xacro:include filename="ros2_control.xacro"/>
 <xacro:include filename="gazebo.xacro"/>
+<!-- Define color materials -->
+<material name="dobot_orange">
+  <color rgba="1.0 0.4 0.0 1.0"/>
+</material>
+<material name="dobot_black">
+  <color rgba="0.2 0.2 0.2 1.0"/>
+</material>
+<material name="dobot_grey">
+  <color rgba="0.6 0.6 0.6 1.0"/>
+</material>
+<material name="dobot_white">
+  <color rgba="0.9 0.9 0.9 1.0"/>
+</material>
  <link name="world"/>
   <link name="base_link">
@@ -24,8 +37,5 @@
         <mesh filename="package://dofbot_description/meshes2/cr5/base_link.dae" />
       </geometry>
-      <material
-        name="">
-        <color rgba="0 0 0 1" />
-      </material>
+      <material name="dobot_black"/>
     </visual>
     <collision>
@@ -58,8 +68,5 @@
         <mesh filename="package://dofbot_description/meshes2/cr5/Link1.dae" />
       </geometry>
-      <material
-        name="">
-        <color rgba="1 1 1 1" />
-      </material>
+      <material name="dobot_orange"/>
     </visual>
     <collision>
@@ -94,8 +101,5 @@
         <mesh filename="package://dofbot_description/meshes2/cr5/Link2.dae" />
       </geometry>
-      <material
-        name="">
-        <color rgba="1 1 1 1" />
-      </material>
+      <material name="dobot_white"/>
     </visual>
     <collision>
@@ -130,8 +134,5 @@
         <mesh filename="package://dofbot_description/meshes2/cr5/Link3.dae" />
       </geometry>
-      <material
-        name="">
-        <color rgba="1 1 1 1" />
-      </material>
+      <material name="dobot_orange"/>
     </visual>
     <collision>
@@ -166,7 +167,5 @@
         <mesh filename="package://dofbot_description/meshes2/cr5/Link4.dae" />
       </geometry>
-      <material name="">
-        <color rgba="1 1 1 1" />
-      </material>
+      <material name="dobot_white"/>
     </visual>
     <collision>
@@ -202,7 +201,5 @@
         <mesh filename="package://dofbot_description/meshes2/cr5/Link5.dae" />
       </geometry>
-      <material name="">
-        <color rgba="1 1 1 1" />
-      </material>
+      <material name="dobot_orange"/>
     </visual>
     <collision>
@@ -237,7 +234,5 @@
         <mesh filename="package://dofbot_description/meshes2/cr5/Link6.dae" />
       </geometry>
-      <material name="">
-        <color rgba="1 1 1 1" />
-      </material>
+      <material name="dobot_black"/>
     </visual>
     <collision>
