Commit message: WIP: Local edits before pulling

File: src/dofbot_description/urdf/new_cr5.xacro (robot description, xacro)
@@ -6,4 +6,5 @@
 <xacro:include filename="ros2_control.xacro"/>
 <xacro:include filename="gazebo.xacro"/>
+ <link name="world"/>
   <link name="base_link">
     <inertial>
@@ -35,5 +36,4 @@
     </collision>
   </link>
-   <link name="world"/>
    <joint name="world_base" type="fixed">
    <parent link="world"/>
@@ -75,5 +75,5 @@
     <child link="Link1" />
     <axis xyz="0 0 1" />
-    <limit lower="-3.14" upper="3.14" effort="0" velocity="0" />
+    <limit lower="-3.14" upper="3.14" effort="100" velocity="10" />
   </joint>
   <link name="Link2">
@@ -111,5 +111,5 @@
     <child  link="Link2" />
     <axis xyz="0 0 1" />
-    <limit lower="-3.14" upper="3.14" effort="0" velocity="0" />
+    <limit lower="-3.14" upper="3.14" effort="100" velocity="10" />
   </joint>
   <link name="Link3">
@@ -147,5 +147,5 @@
     <child link="Link3" />
     <axis  xyz="0 0 1" />
-    <limit lower="-2.86"  upper="2.86"  effort="0" velocity="0" />
+    <limit lower="-2.86"  upper="2.86"  effort="100" velocity="10" />
   </joint>
   <link name="Link4">
@@ -182,5 +182,5 @@
     <child link="Link4" />
     <axis xyz="0 0 1" />
-    <limit lower="-3.14" upper="3.14" effort="0" velocity="0" />
+    <limit lower="-3.14" upper="3.14" effort="100" velocity="10" />
   </joint>
   <link
@@ -218,5 +218,5 @@
     <child link="Link5" />
     <axis xyz="0 0 1" />
-    <limit lower="-3.14" upper="3.14" effort="0" velocity="0" />
+    <limit lower="-3.14" upper="3.14" effort="100" velocity="10" />
   </joint>
   <link name="Link6">
@@ -253,5 +253,5 @@
     <child link="Link6" />
     <axis xyz="0 0 1" />
-    <limit lower="-6.28" upper="6.28" effort="0" velocity="0" />
+    <limit lower="-6.28" upper="6.28" effort="100" velocity="10" />
   </joint>
 </robot>

File: src/dofbot_description/urdf/ros2_control.xacro (robot description, xacro)
@@ -3,10 +3,10 @@
   <ros2_control name="GazeboSystem" type="system">
             <hardware>
-               <plugin>gz_ros2_control/GazeboSimSystem</plugin>
+                <plugin>ign_ros2_control/IgnitionSystem</plugin>
             </hardware>
             <joint name="joint1">
             <command_interface name="position">
-                <param name="min">-1</param>
-                <param name="max">1</param>
+                <!-- <param name="min">-1</param>
+                <param name="max">1</param> -->
             </command_interface>
             <state_interface name="position"/>
@@ -15,6 +15,6 @@
         <joint name="joint2">
             <command_interface name="position">
-                <param name="min">-1</param>
-                <param name="max">1</param>
+                <!-- <param name="min">-1</param>
+                <param name="max">1</param> -->
             </command_interface>
             <state_interface name="position"/>
@@ -23,6 +23,6 @@
         <joint name="joint3">
             <command_interface name="position">
-                <param name="min">-1</param>
-                <param name="max">1</param>
+                <!-- <param name="min">-1</param>
+                <param name="max">1</param> -->
             </command_interface>
             <state_interface name="position"/>
@@ -31,6 +31,6 @@
         <joint name="joint4">
             <command_interface name="position">
-                <param name="min">-1</param>
-                <param name="max">1</param>
+                <!-- <param name="min">-1</param>
+                <param name="max">1</param> -->
             </command_interface>
            <state_interface name="position"/>
@@ -39,6 +39,6 @@
         <joint name="joint5">
             <command_interface name="position">
-                <param name="min">-1</param>
-                <param name="max">1</param>
+                <!-- <param name="min">-1</param>
+                <param name="max">1</param> -->
             </command_interface>
             <state_interface name="position"/>
@@ -47,6 +47,6 @@
         <joint name="joint6">
             <command_interface name="position">
-                <param name="min">-1</param>
-                <param name="max">1</param>
+                <!-- <param name="min">-1</param>
+                <param name="max">1</param> -->
             </command_interface>
             <state_interface name="position"/>
@@ -54,8 +54,3 @@
         </joint>
         </ros2_control>
-<gazebo>
-  <plugin name="gz_ros2_control::GazeboSimROS2ControlPlugin" filename="libgz_ros2_control-system.so">
-            <parameters>$(find dofbot_description)/config/ros2_controllers.yaml</parameters>
-        </plugin>
-</gazebo>
 </robot>

Commit message: added the gripper

File: src/dofbot_description/urdf/new_cr5.xacro (robot description, xacro)
@@ -6,4 +6,5 @@
 <xacro:include filename="ros2_control.xacro"/>
 <xacro:include filename="gazebo.xacro"/>
+<xacro:include filename="gripper.xacro"/>
 <!-- Define color materials -->
 <material name="dobot_orange">

File: src/dofbot_description/urdf/ros2_control.xacro (robot description, xacro)
@@ -47,6 +47,10 @@
         <joint name="joint6">
             <command_interface name="position">
-                <!-- <param name="min">-1</param>
-                <param name="max">1</param> -->
+            </command_interface>
+            <state_interface name="position"/>
+            <state_interface name="velocity"/>
+        </joint>
+        <joint name="robotiq_85_left_knuckle_joint">
+        <command_interface name="position">
             </command_interface>
             <state_interface name="position"/>
