Commit message: fixed gripper controller

File: src/dofbot_description/urdf/gazebo.xacro (robot description, xacro)
@@ -1,26 +1,36 @@
-<?xml version="1.0"?>
+<?xml version="1.0" encoding="utf-8"?>
 <robot xmlns:xacro="http://www.ros.org/wiki/xacro">
    <gazebo reference="base_link">
+        <gravity>false</gravity>
+        <selfCollide>true</selfCollide>
     </gazebo>
     <gazebo reference="Link1">
+        <gravity>false</gravity>
+        <selfCollide>true</selfCollide>
     </gazebo>
     <gazebo reference="Link2">
+        <gravity>false</gravity>
+        <selfCollide>true</selfCollide>
     </gazebo>
     <gazebo reference="Link3">
+        <gravity>false</gravity>
+        <selfCollide>true</selfCollide>
     </gazebo>
     <gazebo reference="Link4">
+        <gravity>false</gravity>
+        <selfCollide>true</selfCollide>
     </gazebo>
     <gazebo reference="Link5">
+        <gravity>false</gravity>
+        <selfCollide>true</selfCollide>
     </gazebo>
     <gazebo reference="Link6">
+        <gravity>false</gravity>
+        <selfCollide>true</selfCollide>
     </gazebo>
-    <gazebo>
-        <!-- ROS 2 Humble -->
-          <plugin filename="ign_ros2_control-system" name="ign_ros2_control::IgnitionROS2ControlPlugin">
-            <parameters>$(find dofbot_description)/config/ros2_controllers.yaml</parameters>
-          </plugin>
-          <plugin filename="libignition-gazebo-sensors-system.so" name="ignition::gazebo::systems::Sensors">
-            <render_engine>ogre2</render_engine>
-          </plugin>
-    </gazebo>
+     <gazebo>
+      <plugin filename="ign_ros2_control-system" name="ign_ros2_control::IgnitionROS2ControlPlugin">
+        <parameters>$(find dofbot_description)/config/ros2_controllers.yaml</parameters>
+      </plugin>
+      </gazebo>
     </robot>

File: src/dofbot_description/urdf/ros2_control.xacro (robot description, xacro)
@@ -57,4 +57,34 @@
             <state_interface name="velocity"/>
         </joint>
+        <joint name="robotiq_85_right_knuckle_joint">
+        <command_interface name="position">
+            </command_interface>
+            <state_interface name="position"/>
+            <state_interface name="velocity"/>
+        </joint>
+        <joint name="robotiq_85_left_inner_knuckle_joint">
+        <command_interface name="position">
+            </command_interface>
+            <state_interface name="position"/>
+            <state_interface name="velocity"/>
+        </joint>
+        <joint name="robotiq_85_left_finger_tip_joint">
+        <command_interface name="position">
+            </command_interface>
+            <state_interface name="position"/>
+            <state_interface name="velocity"/>
+        </joint>
+         <joint name="robotiq_85_right_finger_tip_joint">
+        <command_interface name="position">
+            </command_interface>
+            <state_interface name="position"/>
+            <state_interface name="velocity"/>
+        </joint>
+         <joint name="robotiq_85_right_inner_knuckle_joint">
+        <command_interface name="position">
+            </command_interface>
+            <state_interface name="position"/>
+            <state_interface name="velocity"/>
+        </joint>
         </ros2_control>
 </robot>
